File: HW/rp_nixie/mcu.kicad_sch (KiCad schematic)
At the start: 11 parts, among them J1 PawPad_UART, J2 PawPad_SWD, SW1 RES, U1 PicoW

Commit message: some schematic work
Other:
- moved on the sheet: C5, C6, J1, J2, TP1, TPC1, TPC3
